File: HallSingle/HallSingle.sch (KiCad schematic (older format))
At the start: 10 parts, among them J1 Conn_01x03, U1 SS49E, U2 TS331ILT

Commit message: Updated with revision number. Corrected header orientation. added ibom
Parts:
- added H1: MountingHole, HallEffect:MountingHole_3.2mm_M3, symbol HallEffect:MountingHole
Connections:
- net +5V: now also J1.3 (Pin_3); no longer J1.1 (Pin_1)
- net Signal: now also J1.1 (Pin_1); no longer J1.3 (Pin_3)
Changed lines of the file:
@@
 L power:+5V #PWR09
 U 1 1 5FE9D08F
-P 7300 2200
-F 0 "#PWR09" H 7300 2050 50  0001 C CNN
-F 1 "+5V" V 7315 2328 50  0000 L CNN
-F 2 "" H 7300 2200 50  0001 C CNN
-F 3 "" H 7300 2200 50  0001 C CNN
-	1    7300 2200
+P 7300 2400
+F 0 "#PWR09" H 7300 2250 50  0001 C CNN
+F 1 "+5V" V 7315 2528 50  0000 L CNN
+F 2 "" H 7300 2400 50  0001 C CNN
+F 3 "" H 7300 2400 50  0001 C CNN
+	1    7300 2400
 	0    -1   -1   0
 $EndComp
-Text GLabel 7300 2400 0    50   Input ~ 0
+Text GLabel 7300 2200 0    50   Input ~ 0
 Signal
 $Comp
@@
 Wire Wire Line
 	3100 2150 3100 2200
+$Comp
+L HallEffect:MountingHole H1
+U 1 1 6008E559
+P 6700 3150
+F 0 "H1" H 6800 3196 50  0000 L CNN
+F 1 "MountingHole" H 6800 3105 50  0000 L CNN
+F 2 "HallEffect:MountingHole_3.2mm_M3" H 6700 3150 50  0001 C CNN
+F 3 "~" H 6700 3150 50  0001 C CNN
+	1    6700 3150
+	1    0    0    -1
+$EndComp
 $EndSCHEMATC
