File: HallSingle-TS331/HallSingle.kicad_pcb (KiCad board)
At the start: 2 copper layers, 12 x 23.5 mm, 11 parts, among them J1 Conn_01x03, U1 SS49E, U2 TS331ILT

Commit message: further fixes and gerbers updated this time
Routing:
- net +5V: track 4.36 -> 5.01 mm, vias 3 -> 2
Changed lines of the file:
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@@
   (gr_line (start 150 58) (end 150 79.5) (layer Edge.Cuts) (width 0.05))
   (gr_line (start 139 57) (end 149 57) (layer Edge.Cuts) (width 0.05))
-  (via (at 147.35 58.55) (size 0.8) (drill 0.4) (layers F.Cu B.Cu) (net 4))
   (segment (start 139.554001 58.946999) (end 139.954 58.547) (width 0.3048) (layer F.Cu) (net 1))
   (segment (start 142.2825 59.55) (end 142.272 59.5605) (width 0.6096) (layer F.Cu) (net 1))
@@
   (segment (start 146.558 64.9605) (end 146.558 62.9285) (width 0.3048) (layer F.Cu) (net 2))
   (segment (start 146.4 62.392) (end 146.558 62.55) (width 0.3048) (layer F.Cu) (net 2))
-  (via (at 142.4 63.5) (size 0.8) (drill 0.4) (layers F.Cu B.Cu) (net 3))
-  (via (at 145.25 60.5) (size 0.8) (drill 0.4) (layers F.Cu B.Cu) (net 3))
-  (via (at 139.05 61.45) (size 0.8) (drill 0.4) (layers F.Cu B.Cu) (net 3))
-  (segment (start 139.6 62) (end 139.05 61.45) (width 0.6096) (layer F.Cu) (net 3))
-  (segment (start 139.6 62.3625) (end 139.6 62) (width 0.6096) (layer F.Cu) (net 3))
-  (segment (start 145.1395 60.5105) (end 145.15 60.5) (width 0.6096) (layer F.Cu) (net 3))
-  (segment (start 141.6625 64.2375) (end 142.4 63.5) (width 0.6096) (layer F.Cu) (net 3))
-  (segment (start 141.65 64.2375) (end 141.6625 64.2375) (width 0.6096) (layer F.Cu) (net 3))
-  (segment (start 148 73.5) (end 148 73.6) (width 0.3048) (layer B.Cu) (net 3))
   (segment (start 148.463 60.637) (end 148.6 60.5) (width 0.3048) (layer F.Cu) (net 2))
   (segment (start 148.5 62.3125) (end 148.45 62.3625) (width 0.3048) (layer F.Cu) (net 2))
   (segment (start 148.5 60.45) (end 148.5 62.3125) (width 0.3048) (layer F.Cu) (net 2))
+  (via (at 140.65 63.3) (size 0.8) (drill 0.4) (layers F.Cu B.Cu) (net 3))
+  (via (at 145.25 60.5) (size 0.8) (drill 0.4) (layers F.Cu B.Cu) (net 3))
+  (segment (start 145.1395 60.5105) (end 145.15 60.5) (width 0.6096) (layer F.Cu) (net 3))
+  (segment (start 141.65 64.2375) (end 141.6625 64.2375) (width 0.6096) (layer F.Cu) (net 3))
+  (segment (start 148 73.5) (end 148 73.6) (width 0.3048) (layer B.Cu) (net 3))
   (segment (start 144.2825 60.5) (end 144.272 60.5105) (width 0.6096) (layer F.Cu) (net 3))
   (segment (start 145.25 60.5) (end 144.2825 60.5) (width 0.6096) (layer F.Cu) (net 3))
   (segment (start 145.3 60.45) (end 145.25 60.5) (width 0.6096) (layer F.Cu) (net 3))
   (segment (start 146.3 60.45) (end 145.3 60.45) (width 0.6096) (layer F.Cu) (net 3))
+  (segment (start 139.7125 62.3625) (end 140.65 63.3) (width 0.6096) (layer F.Cu) (net 3))
+  (segment (start 139.6 62.3625) (end 139.7125 62.3625) (width 0.6096) (layer F.Cu) (net 3))
+  (segment (start 140.7125 63.3) (end 141.65 64.2375) (width 0.6096) (layer F.Cu) (net 3))
+  (segment (start 140.65 63.3) (end 140.7125 63.3) (width 0.6096) (layer F.Cu) (net 3))
+  (via (at 147.35 58.55) (size 0.8) (drill 0.4) (layers F.Cu B.Cu) (net 4))
   (via (at 140.9 61.4) (size 0.8) (drill 0.4) (layers F.Cu B.Cu) (net 4))
   (segment (start 141.65 62.3625) (end 141.65 62.15) (width 0.3048) (layer F.Cu) (net 4))
@@
   (segment (start 148 77.82429) (end 149.399999 76.424291) (width 0.3048) (layer B.Cu) (net 4))
   (segment (start 148 78.58) (end 148 77.82429) (width 0.3048) (layer B.Cu) (net 4))
-  (segment (start 143.07763 74) (end 142 74) (width 0.3048) (layer F.Cu) (net 5))
-  (segment (start 148.463 64.613) (end 146.794399 66.281601) (width 0.3048) (layer F.Cu) (net 5))
-  (segment (start 146.794399 66.281601) (end 146.794399 70.283231) (width 0.3048) (layer F.Cu) (net 5))
-  (segment (start 146.794399 70.283231) (end 143.07763 74) (width 0.3048) (layer F.Cu) (net 5))
-  (segment (start 144.5 76.5) (end 142 74) (width 0.3048) (layer F.Cu) (net 5))
   (segment (start 146.451 58.6105) (end 146.4535 58.608) (width 0.3048) (layer F.Cu) (net 4))
   (segment (start 147.35 58.55) (end 146.3 58.55) (width 0.3048) (layer F.Cu) (net 4))
@@
   (segment (start 143.75 58.55) (end 140.9 61.4) (width 0.3048) (layer B.Cu) (net 4))
   (segment (start 147.35 58.55) (end 143.75 58.55) (width 0.3048) (layer B.Cu) (net 4))
+  (segment (start 143.07763 74) (end 142 74) (width 0.3048) (layer F.Cu) (net 5))
+  (segment (start 148.463 64.613) (end 146.794399 66.281601) (width 0.3048) (layer F.Cu) (net 5))
+  (segment (start 146.794399 66.281601) (end 146.794399 70.283231) (width 0.3048) (layer F.Cu) (net 5))
+  (segment (start 146.794399 70.283231) (end 143.07763 74) (width 0.3048) (layer F.Cu) (net 5))
+  (segment (start 144.5 76.5) (end 142 74) (width 0.3048) (layer F.Cu) (net 5))
   (segment (start 144.2825 58.6) (end 144.272 58.6105) (width 0.3048) (layer F.Cu) (net 6))
   (segment (start 147.712689 57.794399) (end 144.383301 57.794399) (width 0.3048) (layer F.Cu) (net 6))
